Commit message: robot update

File: src/diff_drive_robot/urdf/lidar_ray.gazebo.xacro (robot description, xacro)
@@ -8,5 +8,5 @@
           <scan>
             <horizontal>
-              <samples>360</samples>
+              <samples>180</samples>
               <min_angle>-3.14</min_angle>
               <max_angle>3.14</max_angle>

File: src/diff_drive_robot/urdf/robot.gazebo.xacro (robot description, xacro)
@@ -26,5 +26,5 @@
         </plugin>
     </gazebo>
-    <gazebo reference="imu_link">
+    <!-- <gazebo reference="imu_link">
         <sensor name="imu" type="imu">
         <always_on>true</always_on>
@@ -35,5 +35,5 @@
         <gz_frame_id>imu_link</gz_frame_id>
         </sensor>
-    </gazebo>
+    </gazebo> -->
     <!-- Choose one of the following LIDAR sensors by uncommenting the desired lines:  -->
     <!-- <xacro:include filename="$(find diff_drive_robot)/urdf/lidar_gpu.gazebo.xacro"/>

File: src/diff_drive_robot/urdf/robot.urdf (robot description, URDF)
Before this commit: robot diff_drive_robot, 8 links, 7 joints
Links:
- removed link imu_link
Joints:
- removed joint imu_joint
