Commit message: urdf fixed, bridges, amcl, map server working. amcl now waiting for initial pose.

File: src/diff_drive_robot/urdf/lidar_gpu.sensor.xacro (robot description, xacro)
@@ -8,5 +8,5 @@
       <topic>scan</topic>
       <always_on>true</always_on>
-      <!-- <gz_frame_id>laser_frame</gz_frame_id> -->
+      <gz_frame_id>laser</gz_frame_id>
       <ray>
         <scan>

File: src/diff_drive_robot/urdf/robot.gazebo.xacro (robot description, xacro)
@@ -37,10 +37,10 @@
     </gazebo> -->
     <!-- Choose one of the following LIDAR sensors by uncommenting the desired lines:  -->
-    <gazebo reference="laser_frame">
+    <gazebo reference="laser">
         <xacro:include filename="$(find diff_drive_robot)/urdf/lidar_gpu.sensor.xacro"/>
         <xacro:lidar_gpu_sensor/>
     </gazebo>
     <!-- probably never use lidar/ray, since it doesnt work properly for harmonic, while gpu lidar does -->
-    <!-- <gazebo reference="laser_frame">
+    <!-- <gazebo reference="laser">
         <xacro:include filename="$(find diff_drive_robot)/urdf/lidar_ray.sensor.xacro"/>
         <xacro:lidar_ray_sensor/>

File: src/diff_drive_robot/urdf/robot.urdf (robot description, URDF)
Before this commit: robot diff_drive_robot, 7 links, 6 joints
Links:
- removed link laser_frame
- added link laser; collision cylinder length=0.04 radius=0.05; visual cylinder length=0.04 radius=0.05
Joints:
- joint laser_joint: child laser_frame -> laser; parent chassis -> base_link
