Commit message: Fixed LiDAR. Added the option of choosing 180 or 360 LiDAR

File: diff_drive_robot/urdf/lidar_gpu_360_sensor.xacro (robot description, xacro)
@@ -1,5 +1,5 @@
 <?xml version="1.0"?>
 <robot xmlns:xacro="http://www.ros.org/wiki/xacro">
-  <xacro:macro name="lidar_gpu_sensor" params="">
+  <xacro:macro name="lidar_gpu_360_sensor" params="">
     <sensor name="laser" type="gpu_lidar">
       <pose>0 0 0 0 0 0</pose>
@@ -14,6 +14,6 @@
           <!-- if you adapt here make sure to also update the number of beams in the active_inference_loc/models.py -->
             <samples>360</samples>
-            <min_angle>-3.14159</min_angle>   <!-- -180° -->
-            <max_angle> 3.14159</max_angle>   <!-- +180° -->
+            <min_angle>-3.14</min_angle>   <!-- -180° -->
+            <max_angle> 3.14</max_angle>   <!-- +180° -->
           </horizontal>
         </scan>

File: diff_drive_robot/urdf/robot.gazebo.xacro (robot description, xacro)
@@ -37,12 +37,11 @@
     </gazebo> -->
     <!-- Choose one of the following LIDAR sensors by uncommenting the desired lines:  -->
+    <!-- <gazebo reference="laser">
+        <xacro:include filename="$(find diff_drive_robot)/urdf/lidar_gpu_360_sensor.xacro"/>
+        <xacro:lidar_gpu_360_sensor/>
+    </gazebo>  -->
     <gazebo reference="laser">
-        <xacro:include filename="$(find diff_drive_robot)/urdf/lidar_gpu.sensor.xacro"/>
-        <xacro:lidar_gpu_sensor/>
+        <xacro:include filename="$(find diff_drive_robot)/urdf/lidar_gpu_180_sensor.xacro"/>
+        <xacro:lidar_gpu_180_sensor/>
     </gazebo>
-    <!-- probably never use lidar/ray, since it doesnt work properly for harmonic, while gpu lidar does -->
-    <!-- <gazebo reference="laser">
-        <xacro:include filename="$(find diff_drive_robot)/urdf/lidar_ray.sensor.xacro"/>
-        <xacro:lidar_ray_sensor/>
-    </gazebo> -->
 </robot>
